File: parallel2usb_v1/parallel2usb.kicad_sch (KiCad schematic)
At the start: 45 parts, among them J1 DB25_Male_MountingHoles, J2 Conn_01x20, J3 Conn_01x03_Male, U1 74LVC161284DL, U2 Pico

Commit message: Minor schematic and gerber updates.
Connections:
- net JUMPER_PIN: now reaches U2.2 (GPIO1)
Other:
- note added: "2022/12/31"
- note added: "Connect GPIO1 to GND with a jumper to make the firmware print diagnostics to the USB serial port."
- note added: "GPIO28 is floating on the PCB v1, but strapped to GND on v2 to allow firmware to detected the PCB version."
- note added: "Parallel Printer Port to USB Capturing Tool"
- note added: "Parallel2USB"
- note added: "Tom Verbeure https://github.com/tomverbeure/parallel2usb/parallel2usb_v1"
- note added: "v1"
- moved on the sheet: J3, U2
