File: parallel2usb_v2/parallel2usb.kicad_pcb (KiCad board)
At the start: 4 copper layers, 65.3 x 53.6 mm, 45 parts, among them J1 DB25_Male_MountingHoles, J2 Conn_01x20, U1 74LVC161284DL, U2 Pico

Commit message: PCB v2.
Parts:
- removed H1, H2: MountingHole, MountingHole:MountingHole_2.7mm_M2.5
- added C20: 100n, Capacitor_SMD:C_0603_1608Metric_Pad1.08x0.95mm_HandSolder, F.Cu at (177.4, 111.0)
- U2: moved to B.Cu
- moved U2 17.4 mm to (176.5, 101.6), turned to 0 degrees
- moved REF** 15.5 mm to (178.7, 101.7)
- moved R9 6.11 mm to (190.9, 76.1)
- moved R10 5.60 mm to (190.9, 79.1)
- moved C3 5.47 mm to (190.9, 77.6)
- moved R11 5.09 mm to (190.9, 82.2)
- moved C6 5.05 mm to (190.9, 80.6)
- moved C13 4.67 mm to (190.9, 126.4)
- moved C9 4.65 mm to (190.9, 83.7)
- moved R12 4.59 mm to (190.9, 85.2)
- moved C10 4.29 mm to (190.9, 123.3)
- moved C12 4.27 mm to (190.9, 86.7)
- moved R1 4.08 mm to (190.9, 88.3)
- moved C17 3.95 mm to (190.9, 120.3)
- moved C1 3.93 mm to (190.9, 89.8)
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Connections:
- U2 pad 1: unconnected-(U2-Pad1) -> /AUTOF_3
- U2 pad 11: /D3_3 -> /D5_3
- U2 pad 12: /D2_3 -> /D6_3
- U2 pad 14: /D1_3 -> /D7_3
- U2 pad 15: /D0_3 -> /STROBE_3
- U2 pad 16: /SELIN_3 -> /ERROR_3
- U2 pad 17: /INIT_3 -> /ACK_3
- U2 pad 19: /AUTOF_3 -> /BUSY_3
- U2 pad 2: unconnected-(U2-Pad2) -> /INIT_3
- U2 pad 20: /STROBE_3 -> /PE_3
- U2 pad 21: /DIR -> /HD
- U2 pad 22: /HD -> /DIR
- U2 pad 25: /PE_3 -> unconnected-(U2-Pad25)
- U2 pad 26: /BUSY_3 -> unconnected-(U2-Pad26)
- U2 pad 27: /ACK_3 -> unconnected-(U2-Pad27)
- U2 pad 29: /ERROR_3 -> unconnected-(U2-Pad29)
- U2 pad 4: unconnected-(U2-Pad4) -> /SELIN_3
- U2 pad 5: unconnected-(U2-Pad5) -> /D0_3
- U2 pad 6: /D7_3 -> /D1_3
- U2 pad 7: /D6_3 -> /D2_3
- U2 pad 9: /D5_3 -> /D3_3
Routing:
- net GND: track 339.0 -> 281.2 mm, vias 24 -> 9
- net /DIR: track 41.7 -> 16.8 mm
- net +3.3V: track 83.7 -> 63.6 mm
- net +5V: track 83.0 -> 66.0 mm, vias 2 -> 1
- net /STROBE_3: track 37.0 -> 21.1 mm
- net /D6_3: track 21.0 -> 5.61 mm
- net /D7_3: track 23.9 -> 9.02 mm
- net /D0_3: track 26.7 -> 13.2 mm, vias 1 -> 0
- net /AUTOF_3: track 33.8 -> 20.6 mm, vias 2 -> 0
- net /ERROR_3: track 25.0 -> 12.5 mm
- net /D5_3: track 16.9 -> 5.09 mm
- net /ACK_3: track 26.3 -> 14.6 mm
- net /SELIN_3: track 24.9 -> 13.9 mm, vias 2 -> 0
- net /D1_3: track 22.2 -> 11.3 mm, vias 1 -> 0
- net /INIT_3: track 28.0 -> 18.5 mm, vias 2 -> 0
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- added copper zone on B.Cu, net GND
- removed copper zone on In2.Cu, net GND
Other:
- board size 65.3 x 53.6 mm -> 45.1 x 53.6 mm
- copper layers 4 -> 2
- board text added: "AF"
- board text added: "BSY"
- board text added: "ERR"
- board text added: "SELI"
- board text added: "STB"
- board text removed: "AUTOF"
- board text removed: "BUSY"
- board text removed: "ERROR"
- board text removed: "SELINT"
- board text removed: "STROBE"

Commit message: Minor schematic and gerber updates.
Connections:
- U2 pad 27: unconnected-(U2-Pad27) -> /JUMPER_PIN
- U2 pad 34: unconnected-(U2-Pad34) -> GND
Routing:
- net GND: track 281.2 -> 300.4 mm
Changed lines of the file:
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@@
       (drillshape 0)
       (scaleselection 1)
-      (outputdirectory "gerbers/v1/")
+      (outputdirectory "gerbers/v2/")
     )
   )
@@
   (net 56 "unconnected-(U2-Pad31)")
   (net 57 "unconnected-(U2-Pad32)")
-  (net 58 "unconnected-(U2-Pad34)")
+  (net 58 "/JUMPER_PIN")
   (net 59 "unconnected-(U2-Pad35)")
   (net 60 "unconnected-(U2-Pad37)")
@@
   (net 68 "unconnected-(U2-Pad43)")
   (net 69 "unconnected-(U2-Pad26)")
-  (net 70 "unconnected-(U2-Pad27)")
-  (net 71 "unconnected-(U2-Pad29)")
-  (net 72 "unconnected-(U2-Pad25)")
+  (net 70 "unconnected-(U2-Pad29)")
+  (net 71 "unconnected-(U2-Pad25)")
   (footprint "Capacitor_SMD:C_0603_1608Metric_Pad1.08x0.95mm_HandSolder" (layer "F.Cu")
     (at 190.8545 77.597 180)
@@
       (effects (font (size 0.8 0.8) (thickness 0.15)) (justify mirror))
     )
-    (fp_text user "GP21" (at 13.054 -8.9 135) (layer "B.SilkS")
+    (fp_text user "GP21/JP" (at 13.716 -8.001 135) (layer "B.SilkS")
       (effects (font (size 0.8 0.8) (thickness 0.15)) (justify mirror))
     )
-    (fp_text user "GP22" (at 13.054 -3.81 135) (layer "B.SilkS")
+    (fp_text user "GP22" (at 13.081 -3.937 135) (layer "B.SilkS")
       (effects (font (size 0.8 0.8) (thickness 0.15)) (justify mirror))
     )
@@
       (effects (font (size 0.8 0.8) (thickness 0.15)) (justify mirror))
     )
-    (fp_text user "GND" (at 12.8 -6.35 135) (layer "B.SilkS")
+    (fp_text user "GND/JP" (at 13.462 -5.715 135) (layer "B.SilkS")
       (effects (font (size 0.8 0.8) (thickness 0.15)) (justify mirror))
     )
@@
       (net 52 "/SEL_3") (pinfunction "GPIO18") (pintype "bidirectional"))
     (pad "25" smd rect (at 8.89 -13.97) (size 3.5 1.7) (drill (offset 0.9 0)) (layers "B.Cu" "B.Mask")
-      (net 72 "unconnected-(U2-Pad25)") (pinfunction "GPIO19") (pintype "bidirectional+no_connect"))
+      (net 71 "unconnected-(U2-Pad25)") (pinfunction "GPIO19") (pintype "bidirectional+no_connect"))
     (pad "25" thru_hole oval (at 8.89 -13.97) (size 1.7 1.7) (drill 1.02) (layers *.Cu *.Mask)
-      (net 72 "unconnected-(U2-Pad25)") (pinfunction "GPIO19") (pintype "bidirectional+no_connect"))
+      (net 71 "unconnected-(U2-Pad25)") (pinfunction "GPIO19") (pintype "bidirectional+no_connect"))
     (pad "26" smd rect (at 8.89 -11.43) (size 3.5 1.7) (drill (offset 0.9 0)) (layers "B.Cu" "B.Mask")
       (net 69 "unconnected-(U2-Pad26)") (pinfunction "GPIO20") (pintype "bidirectional+no_connect"))
@@
       (net 69 "unconnected-(U2-Pad26)") (pinfunction "GPIO20") (pintype "bidirectional+no_connect"))
     (pad "27" thru_hole oval (at 8.89 -8.89) (size 1.7 1.7) (drill 1.02) (layers *.Cu *.Mask)
-      (net 70 "unconnected-(U2-Pad27)") (pinfunction "GPIO21") (pintype "bidirectional+no_connect"))
+      (net 58 "/JUMPER_PIN") (pinfunction "GPIO21") (pintype "bidirectional+no_connect"))
     (pad "27" smd rect (at 8.89 -8.89) (size 3.5 1.7) (drill (offset 0.9 0)) (layers "B.Cu" "B.Mask")
-      (net 70 "unconnected-(U2-Pad27)") (pinfunction "GPIO21") (pintype "bidirectional+no_connect"))
+      (net 58 "/JUMPER_PIN") (pinfunction "GPIO21") (pintype "bidirectional+no_connect"))
     (pad "28" thru_hole rect (at 8.89 -6.35) (size 1.7 1.7) (drill 1.02) (layers *.Cu *.Mask)
       (net 1 "GND") (pinfunction "GND") (pintype "power_in"))
@@
       (net 1 "GND") (pinfunction "GND") (pintype "power_in"))
     (pad "29" smd rect (at 8.89 -3.81) (size 3.5 1.7) (drill (offset 0.9 0)) (layers "B.Cu" "B.Mask")
-      (net 71 "unconnected-(U2-Pad29)") (pinfunction "GPIO22") (pintype "bidirectional+no_connect"))
+      (net 70 "unconnected-(U2-Pad29)") (pinfunction "GPIO22") (pintype "bidirectional+no_connect"))
     (pad "29" thru_hole oval (at 8.89 -3.81) (size 1.7 1.7) (drill 1.02) (layers *.Cu *.Mask)
-      (net 71 "unconnected-(U2-Pad29)") (pinfunction "GPIO22") (pintype "bidirectional+no_connect"))
+      (net 70 "unconnected-(U2-Pad29)") (pinfunction "GPIO22") (pintype "bidirectional+no_connect"))
     (pad "30" thru_hole oval (at 8.89 -1.27) (size 1.7 1.7) (drill 1.02) (layers *.Cu *.Mask)
       (net 55 "unconnected-(U2-Pad30)") (pinfunction "RUN") (pintype "input+no_connect"))
@@
       (net 1 "GND") (pinfunction "AGND") (pintype "power_in"))
     (pad "34" smd rect (at 8.89 8.89) (size 3.5 1.7) (drill (offset 0.9 0)) (layers "B.Cu" "B.Mask")
-      (net 58 "unconnected-(U2-Pad34)") (pinfunction "GPIO28_ADC2") (pintype "bidirectional+no_connect"))
+      (net 1 "GND") (pinfunction "GPIO28_ADC2") (pintype "bidirectional"))
     (pad "34" thru_hole oval (at 8.89 8.89) (size 1.7 1.7) (drill 1.02) (layers *.Cu *.Mask)
-      (net 58 "unconnected-(U2-Pad34)") (pinfunction "GPIO28_ADC2") (pintype "bidirectional+no_connect"))
+      (net 1 "GND") (pinfunction "GPIO28_ADC2") (pintype "bidirectional"))
     (pad "35" thru_hole oval (at 8.89 11.43) (size 1.7 1.7) (drill 1.02) (layers *.Cu *.Mask)
       (net 59 "unconnected-(U2-Pad35)") (pinfunction "ADC_VREF") (pintype "power_in+no_connect"))
@@
     (effects (font (size 1 1) (thickness 0.15)) (justify mirror))
   )
-  (gr_text "D4" (at 192.532 99.822) (layer "B.SilkS")
+  (gr_text "D4" (at 192.532 100.076) (layer "B.SilkS")
     (effects (font (size 1 1) (thickness 0.15)) (justify mirror))
   )
@@
     (effects (font (size 1 1) (thickness 0.15)) (justify mirror))
   )
-  (gr_text "D5" (at 192.532 97.409) (layer "B.SilkS")
+  (gr_text "D5" (at 192.913 97.028) (layer "B.SilkS")
     (effects (font (size 1 1) (thickness 0.15)) (justify mirror))
   )
@@
     (effects (font (size 1 1) (thickness 0.15)) (justify mirror))
   )
-  (gr_text "D6" (at 192.532 94.869) (layer "B.SilkS")
+  (gr_text "D6" (at 192.913 94.361) (layer "B.SilkS")
     (effects (font (size 1 1) (thickness 0.15)) (justify mirror))
   )
@@
   (segment (start 201.928 102.99) (end 204.216 105.278) (width 0.2) (layer "B.Cu") (net 1))
   (segment (start 196.85 126.873) (end 197.104 127.127) (width 0.2) (layer "B.Cu") (net 1))
+  (segment (start 183.007 109.22) (end 183.007 109.728) (width 0.2) (layer "B.Cu") (net 1))
   (segment (start 168.717 94.173) (end 168.717 93.914) (width 0.2) (layer "B.Cu") (net 1))
   (segment (start 204.216 103.124) (end 204.216 99.949) (width 0.2) (layer "B.Cu") (net 1))
@@
   (segment (start 180.467 120.65) (end 179.451 119.634) (width 0.2) (layer "B.Cu") (net 1))
   (segment (start 179.451 109.601) (end 179.832 109.22) (width 0.2) (layer "B.Cu") (net 1))
+  (segment (start 180.086 83.82) (end 181.356 82.55) (width 0.2) (layer "B.Cu") (net 1))
   (segment (start 180.721 100.33) (end 180.721 94.615) (width 0.2) (layer "B.Cu") (net 1))
   (segment (start 179.324 110.998) (end 179.451 111.125) (width 0.2) (layer "B.Cu") (net 1))
@@
   (segment (start 204.216 97.282) (end 204.216 94.234) (width 0.2) (layer "B.Cu") (net 1))
   (segment (start 201.928 89.14) (end 204.216 91.428) (width 0.2) (layer "B.Cu") (net 1))
+  (segment (start 183.769 110.49) (end 185.42 110.49) (width 0.2) (layer "B.Cu") (net 1))
   (segment (start 180.086 93.98) (end 180.721 94.615) (width 0.2) (layer "B.Cu") (net 1))
   (segment (start 204.216 89.027) (end 204.216 81.763) (width 0.2) (layer "B.Cu") (net 1))
@@
   (segment (start 201.928 100.22) (end 204.216 102.508) (width 0.2) (layer "B.Cu") (net 1))
   (segment (start 204.216 121.447) (end 204.216 108.458) (width 0.2) (layer "B.Cu") (net 1))
+  (segment (start 181.356 82.55) (end 185.42 82.55) (width 0.2) (layer "B.Cu") (net 1))
   (segment (start 204.216 99.738) (end 204.216 99.949) (width 0.2) (layer "B.Cu") (net 1))
+  (segment (start 183.007 109.728) (end 183.769 110.49) (width 0.2) (layer "B.Cu") (net 1))
   (segment (start 196.469 125.349) (end 196.85 125.73) (width 0.2) (layer "B.Cu") (net 1))
   (segment (start 201.928 86.37) (end 204.216 88.658) (width 0.2) (layer "B.Cu") (net 1))
@@
   (segment (start 168.717 109.027) (end 167.64 107.95) (width 0.2) (layer "B.Cu") (net 1))
   (segment (start 200.508 125.155) (end 204.216 121.447) (width 0.2) (layer "B.Cu") (net 1))
+  (segment (start 180.086 93.98) (end 180.086 83.82) (width 0.2) (layer "B.Cu") (net 1))
   (segment (start 204.216 81.763) (end 200.508 78.055) (width 0.2) (layer "B.Cu") (net 1))
   (segment (start 204.216 105.278) (end 204.216 105.664) (width 0.2) (layer "B.Cu") (net 1))
