File: parallel2usb_v2/parallel2usb.kicad_sch (KiCad schematic)
At the start: 44 parts, among them J1 DB25_Male_MountingHoles, J2 Conn_01x20, U1 74LVC161284DL, U2 Pico

Commit message: PCB v2.
Parts:
- removed C19: 22u, Capacitor_SMD:C_0603_1608Metric_Pad1.08x0.95mm_HandSolder, symbol Device:C_Polarized
- removed H1, H2: MountingHole, MountingHole:MountingHole_2.7mm_M2.5, symbol Mechanical:MountingHole
- added C19: 22u, Capacitor_SMD:C_0603_1608Metric_Pad1.08x0.95mm_HandSolder, symbol Device:C
- added C20: 100n, Capacitor_SMD:C_0603_1608Metric_Pad1.08x0.95mm_HandSolder, symbol Device:C
Connections:
- net +3.3V: now also C19.1
- net +5V: now also C20.1
- net ACK_3: now also U2.17 (GPIO13); no longer U2.27 (GPIO21)
- net AUTOF_3: now also U2.1 (GPIO0); no longer U2.19 (GPIO14)
- net BUSY_3: now also U2.19 (GPIO14); no longer U2.26 (GPIO20)
- net D0_3: now also U2.5 (GPIO3); no longer U2.15 (GPIO11)
- net D1_3: now also U2.6 (GPIO4); no longer U2.14 (GPIO10)
- net D2_3: now also U2.7 (GPIO5); no longer U2.12 (GPIO9)
- net D3_3: now also U2.9 (GPIO6); no longer U2.11 (GPIO8)
- net D5_3: now also U2.11 (GPIO8); no longer U2.9 (GPIO6)
- net D6_3: now also U2.12 (GPIO9); no longer U2.7 (GPIO5)
- net D7_3: now also U2.14 (GPIO10); no longer U2.6 (GPIO4)
- net DIR: now also U2.22 (GPIO17); no longer U2.21 (GPIO16)
- net ERROR_3: now also U2.16 (GPIO12); no longer U2.29 (GPIO22)
- net GND: now also C19.2, C20.2
- net HD: now also U2.21 (GPIO16); no longer U2.22 (GPIO17)
- net INIT_3: now also U2.2 (GPIO1); no longer U2.17 (GPIO13)
- net PE_3: now also U2.20 (GPIO15); no longer U2.25 (GPIO19)
- net SELIN_3: now also U2.4 (GPIO2); no longer U2.16 (GPIO12)
- net STROBE_3: now also U2.15 (GPIO11); no longer U2.20 (GPIO15)
Other:
- note added: "2023/1/16"
- note added: "Parallel Printer Port to USB Capturing Tool"
- note added: "Parallel2USB"
- note added: "Tom Verbeure https://github.com/tomverbeure/parallel2usb"
- note added: "v2"

Commit message: Minor schematic and gerber updates.
Connections:
- net GND: now also U2.34 (GPIO28_ADC2)
- net JUMPER_PIN: now reaches U2.27 (GPIO21)
- no-connect marks 16 -> 15
Other:
- note added: "Connect GPIO21 to GND with a jumper to make the firmware print diagnostics to the USB serial port."
- note added: "GPIO28 strapped to ground to allow board revision detection in firmware."
- note added: "Tom Verbeure https://github.com/tomverbeure/parallel2usb/parallel2usb_v2"
- note removed: "Tom Verbeure https://github.com/tomverbeure/parallel2usb"
- moved on the sheet: U2
